Commit message: add stl model

File: models/airstand/platform/platform.urdf (robot description, URDF)
Before this commit: robot platform, 1 links, 0 joints
Links:
- link base_link: geometry collision cylinder length=0.49 radius=0.15; visual mesh filename=file:///home/lab1/Projects/airstand/ros/simvis/models/airst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 scale=0.01 0.01 0.01

File: models/airstand/platform/platform.urdf.xacro (robot description, xacro)
@@ -2,21 +2,20 @@
 <robot xmlns:xacro="http://www.ros.org/wiki/xacro" name="platform">
 <xacro:include filename="$(env MODELS_DIR)/common/utils.xacro" />
-<xacro:property name="base_height" value="0.07" />
+<xacro:property name="base_height" value="0.49" />
 <xacro:property name="base_radius" value="0.15" />
-<xacro:property name="prof_height" value="0.4" />
-<xacro:property name="prof_radius" value="0.03" />
 <link name="base_link">
-    <xacro:primitive name="base">
-        <origin xyz="0 0 ${base_height / 2}" rpy="0 0 0" />
+    <visual name="base">
+        <origin xyz="0 0 0" rpy="0 0 0" />
+        <geometry>
+            <mesh
+                filename="file:///home/lab1/Projects/airstand/ros/simvis/models/airstand/platform/platform.stl"
+                scale="0.01 0.01 0.01"
+            />
+        </geometry>
+    </visual>
+    <collision name="base">
+        <origin xyz="0 0 0" rpy="0 0 0" />
         <geometry><cylinder length="${base_height}" radius="${base_radius}"/></geometry>
-    </xacro:primitive>
-    <xacro:primitive name="prof">
-        <origin xyz="0 0 ${base_height + prof_height / 2}" rpy="0 0 0" />
-        <geometry><cylinder length="${prof_height}" radius="${prof_radius}"/></geometry>
-    </xacro:primitive>
-    <xacro:primitive name="plate">
-        <origin xyz="0 0 ${base_height + prof_height}" rpy="0 0 0" />
-        <geometry><box size="0.21 0.297 0.01"/></geometry>
-    </xacro:primitive>
+    </collision>
     <inertial>
         <origin rpy="0 0 0" xyz="0 0 1.0"/>
