Commit message: initirt plane

File: models/airstand/platform/platform.sdf.xacro (robot description, xacro)
@@ -4,6 +4,4 @@
 <xacro:include filename="$(env MODELS_DIR)/common/utils.xacro" />
 <xacro:include filename="propeller.xacro" />
-<xacro:property name="base_height" value="0.59" />
-<xacro:property name="base_radius" value="0.15" />
 <link name="base">
     <visual name="base_visual">

File: models/common/utils.xacro (robot description, xacro)
@@ -1,3 +1,5 @@
 <include xmlns:xacro="http://www.ros.org/wiki/xacro">
+<xacro:property name="base_height" value="0.59" />
+<xacro:property name="base_radius" value="0.15" />
 <xacro:macro name="primitive" params="name *origin *geometry">
   <visual name="${name}">
