Commit message: Correct propellers

File: models/airstand/platform/propeller.xacro (robot description, xacro)
@@ -1,15 +1,21 @@
 <include xmlns:xacro="http://www.ros.org/wiki/xacro">
 <xacro:macro name="propeller" params="name side">
+<xacro:if value="${side == 1}">
+    <xacro:property name="motor_number" value="0" />
+</xacro:if>
+<xacro:if value="${side != 1}">
+    <xacro:property name="motor_number" value="1" />
+</xacro:if>
 <link name="${name}">
     <pose relative_to='base'>0 ${side * 0.17} ${-base_height/2 + 0.165} 0 0 0</pose>
     <inertial>
-        <mass>0.1</mass>
+        <mass>0.04</mass>
         <inertia>
-            <ixx>0.334</ixx>
+            <ixx>0.0001</ixx>
             <ixy>0</ixy>
             <ixz>0</ixz>
-            <iyy>0.334</iyy>
+            <iyy>0.00007</iyy>
             <iyz>0</iyz>
-            <izz>0.0017</izz>
+            <izz>0.00006</izz>
         </inertia>
     </inertial>
@@ -34,7 +40,9 @@
   name="gz::sim::systems::Thruster">
   <joint_name>${name}_joint</joint_name>
-  <thrust_coefficient>1</thrust_coefficient>
+  <use_angvel_cmd>true</use_angvel_cmd>
+  <thrust_coefficient>0.001</thrust_coefficient>
   <fluid_density>1.225</fluid_density>
   <propeller_diameter>0.2</propeller_diameter>
+  <velocity_control>false</velocity_control>
   <p_gain>0</p_gain>
   <d_gain>0</d_gain>
