Commit message: fully integrated gazebo and rviz

File: models/airstand/platform/platform.urdf.xacro (robot description, xacro)
@@ -21,4 +21,6 @@
         </geometry>
     </collision>
+</link>
+<link name="base_weight">
     <inertial>
         <mass value="3.3" />
@@ -26,4 +28,8 @@
     </inertial>
 </link>
+<joint name="base_weight_joint" type="fixed">
+    <parent link="base"/>
+    <child link="base_weight"/>
+</joint>
 <gazebo>
     <plugin

Commit message: Add IMU

File: models/airstand/platform/platform.urdf.xacro (robot description, xacro)
@@ -32,4 +32,11 @@
     <child link="base_weight"/>
 </joint>
+<link name="imu">
+</link>
+<joint name="imu_joint" type="fixed">
+    <parent link="base"/>
+    <child link="imu"/>
+    <origin xyz="0 0 ${base_height/2}"/>
+</joint>
 <gazebo>
     <plugin
@@ -41,4 +48,13 @@
   </plugin>
 </gazebo>
+<gazebo reference="imu">
+    <sensor name="imu" type="imu">
+        <always_on>1</always_on>
+        <update_rate>100</update_rate>
+        <visualize>true</visualize>
+        <topic>imu</topic>
+        <enable_metrics>true</enable_metrics>
+    </sensor>
+</gazebo>
 <xacro:propeller name="prop_left" side="1"/>
 <xacro:propeller name="prop_right" side="-1"/>

File: models/airstand/plugins.xacro (robot description, xacro)
@@ -16,3 +16,6 @@
     <real_time_factor>1.0</real_time_factor>
 </physics>
+<plugin filename="gz-sim-imu-system"
+        name="gz::sim::systems::Imu">
+</plugin>
 </include>

Commit message: add camera

File: models/airstand/platform/platform.urdf.xacro (robot description, xacro)
@@ -32,6 +32,5 @@
     <child link="base_weight"/>
 </joint>
-<link name="imu">
-</link>
+<link name="imu"></link>
 <joint name="imu_joint" type="fixed">
     <parent link="base"/>
@@ -39,4 +38,38 @@
     <origin xyz="0 0 ${base_height/2}"/>
 </joint>
+<gazebo reference="imu">
+    <sensor name="imu" type="imu">
+        <always_on>1</always_on>
+        <update_rate>100</update_rate>
+        <visualize>true</visualize>
+        <topic>imu</topic>
+        <enable_metrics>true</enable_metrics>
+    </sensor>
+</gazebo>
+<link name="camera"></link>
+<joint name="camera_joint" type="fixed">
+    <parent link="base"/>
+    <child link="camera"/>
+    <origin xyz="0 0 ${base_height/2 + 0.02}"/>
+</joint>
+<gazebo reference="camera">
+    <sensor name="camera" type="camera">
+        <camera>
+            <horizontal_fov>1.047</horizontal_fov>
+            <image>
+                <width>320</width>
+                <height>240</height>
+            </image>
+            <clip>
+                <near>0.1</near>
+                <far>100</far>
+            </clip>
+        </camera>
+        <always_on>1</always_on>
+        <update_rate>30</update_rate>
+        <visualize>true</visualize>
+        <topic>camera</topic>
+    </sensor>
+</gazebo>
 <gazebo>
     <plugin
@@ -48,13 +81,4 @@
   </plugin>
 </gazebo>
-<gazebo reference="imu">
-    <sensor name="imu" type="imu">
-        <always_on>1</always_on>
-        <update_rate>100</update_rate>
-        <visualize>true</visualize>
-        <topic>imu</topic>
-        <enable_metrics>true</enable_metrics>
-    </sensor>
-</gazebo>
 <xacro:propeller name="prop_left" side="1"/>
 <xacro:propeller name="prop_right" side="-1"/>

File: models/airstand/plugins.xacro (robot description, xacro)
@@ -19,3 +19,7 @@
         name="gz::sim::systems::Imu">
 </plugin>
+<plugin filename="gz-sim-sensors-system"
+        name="gz::sim::systems::Sensors">
+    <render_engine>ogre2</render_engine>
+</plugin>
 </include>

Commit message: simple flyer model

File: models/airstand/platform/platform.urdf.xacro (robot description, xacro)
@@ -2,5 +2,4 @@
 <robot name="platform" xmlns:xacro="http://www.ros.org/wiki/xacro">
 <xacro:include filename="$(env MODELS_DIR)/common/utils.xacro" />
-<xacro:include filename="propeller.xacro" />
 <link name="base">
     <visual name="base_visual">
@@ -43,43 +42,7 @@
         <update_rate>100</update_rate>
         <visualize>true</visualize>
-        <topic>imu</topic>
+        <topic>platofrm/imu</topic>
         <enable_metrics>true</enable_metrics>
     </sensor>
 </gazebo>
-<link name="camera"></link>
-<joint name="camera_joint" type="fixed">
-    <parent link="base"/>
-    <child link="camera"/>
-    <origin xyz="0 0 ${base_height/2 + 0.02}"/>
-</joint>
-<gazebo reference="camera">
-    <sensor name="camera" type="camera">
-        <camera>
-            <horizontal_fov>1.047</horizontal_fov>
-            <image>
-                <width>320</width>
-                <height>240</height>
-            </image>
-            <clip>
-                <near>0.1</near>
-                <far>100</far>
-            </clip>
-        </camera>
-        <always_on>1</always_on>
-        <update_rate>30</update_rate>
-        <visualize>true</visualize>
-        <topic>camera</topic>
-    </sensor>
-</gazebo>
-<gazebo>
-    <plugin
-        filename="gz-sim-joint-state-publisher-system"
-        name="gz::sim::systems::JointStatePublisher">
-        <topic>joint_states</topic> <!--from <ros><remapping> -->
-        <joint_name>prop_left_joint</joint_name>
-        <joint_name>prop_right_joint</joint_name>
-  </plugin>
-</gazebo>
-<xacro:propeller name="prop_left" side="1"/>
-<xacro:propeller name="prop_right" side="-1"/>
 </robot>

File: models/flyer/flyer.urdf.xacro (robot description, xacro)
@@ -5,5 +5,5 @@
 <link name="base">
     <visual name="base_visual">
-        <origin  xyz="0 ${-robot_side_len/2} 0"/>
+        <origin  xyz="0 0 ${-robot_side_len/2}" rpy="${pi / 2} 0 ${pi / 2}"/>
         <geometry>
             <mesh
@@ -27,4 +27,12 @@
         <inertia ixx="${robot_mass/6}" ixy="0" ixz="0" iyy="${robot_mass/6}" iyz="0" izz="${robot_mass/6}"/>
     </inertial>
+    <visual name="base_visual">
+        <geometry>
+            <sphere radius="0.08"/>
+            <material name="red">
+                <color rgba="1.0 0 0 1.0"/>
+            </material>
+        </geometry>
+    </visual>
 </link>
 <joint name="base_weight_joint" type="fixed">
@@ -32,3 +40,57 @@
     <child link="base_weight"/>
 </joint>
+<!-- IMU BLOCK-->
+<link name="imu"></link>
+<joint name="imu_joint" type="fixed">
+    <parent link="base"/>
+    <child link="imu"/>
+</joint>
+<gazebo reference="imu">
+    <sensor name="imu" type="imu">
+        <always_on>1</always_on>
+        <update_rate>100</update_rate>
+        <visualize>true</visualize>
+        <topic>imu</topic>
+        <enable_metrics>true</enable_metrics>
+    </sensor>
+</gazebo>
+<!-- END IMU BLOCK-->
+<!-- CAMERA BLOCK-->
+<link name="camera"></link>
+<joint name="camera_joint" type="fixed">
+    <parent link="base"/>
+    <child link="camera"/>
+    <origin xyz="0 0 ${robot_side_len/2}"/>
+</joint>
+<gazebo reference="camera">
+    <sensor name="camera" type="camera">
+        <camera>
+            <horizontal_fov>1.047</horizontal_fov>
+            <image>
+                <width>320</width>
+                <height>240</height>
+            </image>
+            <clip>
+                <near>0.1</near>
+                <far>100</far>
+            </clip>
+        </camera>
+        <always_on>1</always_on>
+        <update_rate>30</update_rate>
+        <visualize>true</visualize>
+        <topic>camera</topic>
+    </sensor>
+</gazebo>
+<!-- END CAMERA BLOCK-->
+<gazebo>
+    <plugin
+        filename="gz-sim-joint-state-publisher-system"
+        name="gz::sim::systems::JointStatePublisher">
+        <topic>joint_states</topic> <!--from <ros><remapping> -->
+        <joint_name>prop_bl_joint</joint_name>
+        <joint_name>prop_fl_joint</joint_name>
+  </plugin>
+</gazebo>
+<xacro:propeller name="prop_fl" xyz="${robot_side_len / 2 + 0.05} 0 0" rpy="0 0 0"/>
+<xacro:propeller name="prop_bl" xyz="${-robot_side_len / 2 - 0.05} 0 0" rpy="0 0 ${pi}"/>
 </robot>

File: models/flyer/propeller.xacro (robot description, xacro)
@@ -1,10 +1,4 @@
 <include xmlns:xacro="http://www.ros.org/wiki/xacro">
-<xacro:macro name="propeller" params="name side">
-<xacro:if value="${side == 1}">
-    <xacro:property name="motor_number" value="0" />
-</xacro:if>
-<xacro:if value="${side != 1}">
-    <xacro:property name="motor_number" value="1" />
-</xacro:if>
+<xacro:macro name="propeller" params="name xyz rpy">
 <link name="${name}">
     <inertial>
@@ -16,11 +10,11 @@
             <box size="0.01 0.1 0.1"/>
         </geometry>
-        <material name="red">
-            <color rgba="1.0 0 0 1.0"/>
+        <material name="green">
+            <color rgba="0 1.0 0 1.0"/>
         </material>
     </visual>
 </link>
 <joint name="${name}_joint" type="revolute">
-    <origin xyz="0 ${side * 0.17} ${-base_height/2 + 0.165}"/>
+    <origin xyz="${xyz}" rpy="${rpy}"/>
     <parent link="base"/>
     <child link="${name}"/>
