Commit message: roslaunch gazebo and rviz

File: models/airstand/infinistand.sdf.xacro (robot description, xacro)
@@ -11,8 +11,4 @@
         <xacro:glass_plate z="-0.01" w="100" l="100" thickness="0.02"/>
         </model>
-        <include>
-            <uri>airstand/platform</uri>
-            <pose>0 0 ${base_height / 2} 0 0 0</pose>
-        </include>
     </world>
 </sdf>

File: models/airstand/platform/propeller.xacro (robot description, xacro)
@@ -8,45 +8,39 @@
 </xacro:if>
 <link name="${name}">
-    <pose relative_to='base'>0 ${side * 0.17} ${-base_height/2 + 0.165} 0 0 0</pose>
     <inertial>
-        <mass>0.04</mass>
-        <inertia>
-            <ixx>0.0001</ixx>
-            <ixy>0</ixy>
-            <ixz>0</ixz>
-            <iyy>0.00007</iyy>
-            <iyz>0</iyz>
-            <izz>0.00006</izz>
-        </inertia>
+        <mass value="0.04" />
+        <inertia ixx="0.0001" ixy="0" ixz="0" iyy="0.00007" iyz="0" izz="0.00006"/>
     </inertial>
     <visual name="prop_${name}_vis">
-        <geometry><box>
-            <size>0.01 0.1 0.1</size>
-        </box></geometry>
-        <material>
-            <diffuse>1 0 0</diffuse>
+        <geometry>
+            <box size="0.01 0.1 0.1"/>
+        </geometry>
+        <material name="red">
+            <color rgba="1.0 0 0 1.0"/>
         </material>
     </visual>
 </link>
 <joint name="${name}_joint" type="revolute">
-    <parent>base</parent>
-    <child>${name}</child>
-    <axis>
-        <xyz>1 0 0</xyz>
-    </axis>
+    <origin xyz="0 ${side * 0.17} ${-base_height/2 + 0.165}"/>
+    <parent link="base"/>
+    <child link="${name}"/>
+    <axis xyz="1 0 0"/>
+    <limit effort="100" velocity="100"/>
 </joint>
-<plugin
-  filename="gz-sim-thruster-system"
-  name="gz::sim::systems::Thruster">
-  <joint_name>${name}_joint</joint_name>
-  <use_angvel_cmd>true</use_angvel_cmd>
-  <thrust_coefficient>0.001</thrust_coefficient>
-  <fluid_density>1.225</fluid_density>
-  <propeller_diameter>0.2</propeller_diameter>
-  <velocity_control>false</velocity_control>
-  <p_gain>0</p_gain>
-  <d_gain>0</d_gain>
-  <i_gain>0</i_gain>
-</plugin>
+<gazebo>
+    <plugin
+        filename="gz-sim-thruster-system"
+        name="gz::sim::systems::Thruster">
+        <joint_name>${name}_joint</joint_name>
+        <use_angvel_cmd>true</use_angvel_cmd>
+        <thrust_coefficient>0.001</thrust_coefficient>
+        <fluid_density>1.225</fluid_density>
+        <propeller_diameter>0.2</propeller_diameter>
+        <velocity_control>false</velocity_control>
+        <p_gain>0</p_gain>
+        <d_gain>0</d_gain>
+        <i_gain>0</i_gain>
+    </plugin>
+</gazebo>
 </xacro:macro>
 </include>
