Commit message: add initial flyer model

File: models/common/utils.xacro (robot description, xacro)
@@ -2,4 +2,6 @@
 <xacro:property name="base_height" value="0.59" />
 <xacro:property name="base_radius" value="0.15" />
+<xacro:property name="robot_side_len" value="0.2" />
+<xacro:property name="robot_mass" value="2" />
 <xacro:macro name="primitive" params="name *origin *geometry">
   <visual name="${name}">

Commit message: joined platform and model

File: models/common/utils.xacro (robot description, xacro)
@@ -1,4 +1,4 @@
 <include xmlns:xacro="http://www.ros.org/wiki/xacro">
-<xacro:property name="base_height" value="0.59" />
+<xacro:property name="base_height" value="0.655" />
 <xacro:property name="base_radius" value="0.15" />
 <xacro:property name="robot_side_len" value="0.2" />

File: models/flyer/flyer.urdf.xacro (robot description, xacro)
@@ -1,96 +1,5 @@
 <?xml version="1.0"?>
-<robot name="platform" xmlns:xacro="http://www.ros.org/wiki/xacro">
-<xacro:include filename="$(env MODELS_DIR)/common/utils.xacro" />
-<xacro:include filename="propeller.xacro" />
-<link name="base">
-    <visual name="base_visual">
-        <origin  xyz="0 0 ${-robot_side_len/2}" rpy="${pi / 2} 0 ${pi / 2}"/>
-        <geometry>
-            <mesh
-                filename="file:///$(env MODELS_DIR)/flyer/Astro_m.stl"
-            />
-        </geometry>
-        <material name="blue">
-            <color rgba="0 0 0.7 1.0"/>
-        </material>
-    </visual>
-    <collision name="base_collision">
-        <origin  xyz="0 0 0"/>
-        <geometry>
-            <box size="${robot_side_len} ${robot_side_len} ${robot_side_len}" />
-        </geometry>
-    </collision>
-</link>
-<link name="base_weight">
-    <inertial>
-        <mass value="${robot_mass}" />
-        <inertia ixx="${robot_mass/6}" ixy="0" ixz="0" iyy="${robot_mass/6}" iyz="0" izz="${robot_mass/6}"/>
-    </inertial>
-    <visual name="base_visual">
-        <geometry>
-            <sphere radius="0.08"/>
-            <material name="red">
-                <color rgba="1.0 0 0 1.0"/>
-            </material>
-        </geometry>
-    </visual>
-</link>
-<joint name="base_weight_joint" type="fixed">
-    <parent link="base"/>
-    <child link="base_weight"/>
-</joint>
-<!-- IMU BLOCK-->
-<link name="imu"></link>
-<joint name="imu_joint" type="fixed">
-    <parent link="base"/>
-    <child link="imu"/>
-</joint>
-<gazebo reference="imu">
-    <sensor name="imu" type="imu">
-        <always_on>1</always_on>
-        <update_rate>100</update_rate>
-        <visualize>true</visualize>
-        <topic>imu</topic>
-        <enable_metrics>true</enable_metrics>
-    </sensor>
-</gazebo>
-<!-- END IMU BLOCK-->
-<!-- CAMERA BLOCK-->
-<link name="camera"></link>
-<joint name="camera_joint" type="fixed">
-    <parent link="base"/>
-    <child link="camera"/>
-    <origin xyz="0 0 ${robot_side_len/2}"/>
-</joint>
-<gazebo reference="camera">
-    <sensor name="camera" type="camera">
-        <camera>
-            <horizontal_fov>1.047</horizontal_fov>
-            <image>
-                <width>320</width>
-                <height>240</height>
-            </image>
-            <clip>
-                <near>0.1</near>
-                <far>100</far>
-            </clip>
-        </camera>
-        <always_on>1</always_on>
-        <update_rate>30</update_rate>
-        <visualize>true</visualize>
-        <topic>camera</topic>
-    </sensor>
-</gazebo>
-<!-- END CAMERA BLOCK-->
-<gazebo>
-    <plugin
-        filename="gz-sim-joint-state-publisher-system"
-        name="gz::sim::systems::JointStatePublisher">
-        <topic>joint_states</topic> <!--from <ros><remapping> -->
-        <joint_name>prop_bl_joint</joint_name>
-        <joint_name>prop_fl_joint</joint_name>
-  </plugin>
-</gazebo>
-<xacro:propeller name="prop_fl" xyz="${robot_side_len / 2 + 0.05} 0 0" rpy="0 0 0"/>
-<xacro:propeller name="prop_bl" xyz="${-robot_side_len / 2 - 0.05} 0 0" rpy="0 0 ${pi}"/>
+<robot name="flyer" xmlns:xacro="http://www.ros.org/wiki/xacro">
+<xacro:include filename="$(env MODELS_DIR)/flyer/flyer.xacro" />
+<xacro:flyer/>
 </robot>

File: models/flyer/propeller.xacro (robot description, xacro)
@@ -8,5 +8,5 @@
     <visual name="prop_${name}_vis">
         <geometry>
-            <box size="0.01 0.1 0.1"/>
+            <box size="0.01 0.05 0.05"/>
         </geometry>
         <material name="green">
@@ -27,5 +27,5 @@
         name="gz::sim::systems::Thruster">
         <joint_name>${name}_joint</joint_name>
-        <thrust_coefficient>0.001</thrust_coefficient>
+        <thrust_coefficient>1.0</thrust_coefficient>
         <fluid_density>1.225</fluid_density>
         <propeller_diameter>0.2</propeller_diameter>

File: models/worlds/glass.xacro (robot description, xacro)
@@ -12,6 +12,6 @@
             <friction>
             <ode>
-                <mu>0.0005</mu>
-                <mu2>0.0005</mu2>
+                <mu>0.0045</mu>
+                <mu2>0.0045</mu2>
             </ode>
             </friction>
@@ -25,8 +25,8 @@
         </geometry>
         <material>
-            <diffuse>0.5 0.5 0.5</diffuse>
+            <diffuse>1.0 1.0 1.0</diffuse>
             <script>
                 <uri>file://media/materials/scripts/gazebo.material</uri>
-                <name>Gazebo/Grey</name>
+                <name>Gazebo/White</name>
             </script>
         </material>

File: models/worlds/infinistand.sdf.xacro (robot description, xacro)
@@ -8,6 +8,6 @@
         <xacro:include filename="./glass.xacro" />
         <model name="Glass">
-        <static>true</static>
-        <xacro:glass_plate z="-0.01" w="100" l="100" thickness="0.02"/>
+            <static>true</static>
+            <xacro:glass_plate z="-0.01" w="100" l="100" thickness="0.02"/>
         </model>
     </world>

Commit message: update structure

File: models/common/utils.xacro (robot description, xacro)
@@ -1,16 +1,39 @@
 <include xmlns:xacro="http://www.ros.org/wiki/xacro">
-<xacro:property name="base_height" value="0.655" />
-<xacro:property name="base_radius" value="0.15" />
-<xacro:property name="robot_side_len" value="0.2" />
-<xacro:property name="robot_mass" value="2" />
-<xacro:macro name="primitive" params="name *origin *geometry">
-  <visual name="${name}">
-    <xacro:insert_block name="origin"/>
-    <xacro:insert_block name="geometry"/>
+<xacro:property
+  name="gazebo_systems_lib_dir"
+  value="$(env PROJECT_ROOT)/install/gazebo_systems/lib/gazebo_systems"
+/>
+<xacro:macro name="cuboid_form" params="a b c">
+    <geometry>
+      <box size="${a} ${b} ${c}"/>
+    </geometry>
+</xacro:macro>
+<xacro:macro name="cuboid_inertia" params="weight a b c xyz:='0 0 0' rpy:='0 0 0'">
+  <inertial>
+    <origin xyz="${xyz}" rpy="${rpy}" />
+    <mass value="${weight}" />
+    <inertia ixx="${weight * (a**2 + c**2) / 12}" ixy="0" ixz="0" iyy="${weight * (b**2 + c**2) / 12}" iyz="0" izz="${weight * (b**2 + a**2) / 12}"/>
+  </inertial>
+</xacro:macro>
+<!-- TODO: update to urdf-->
+<xacro:macro name="cuboid" params="name a b c weight pose:='0 0 0 0 0 0' color:=Yellow is_kinematic:=false self_collide:=false">
+<link name="${name}">
+  <self_collide>${self_collide}</self_collide>
+  <kinematic>${is_kinematic}</kinematic>
+  <pose>${pose}</pose>
+  <collision name="${name}_collision">
+    <xacro:cuboid_form a="${a}" b="${b}" c="${c}"/>
+  </collision>
+  <visual name="${name}_visual">
+    <xacro:cuboid_form a="${a}" b="${b}" c="${c}"/>
+    <material>
+      <script>
+          <uri>file://media/materials/scripts/gazebo.material</uri>
+          <name>Gazebo/${color}</name>
+      </script>
+    </material>
   </visual>
-  <collision name="${name}">
-    <xacro:insert_block name="origin"/>
-    <xacro:insert_block name="geometry"/>
-  </collision>
+  <xacro:cuboid_inertia weight="${weight}" a="${a}" b="${b}" c="${c}"/>
+</link>
 </xacro:macro>
 </include>

File: models/flyer/flyer.xacro (robot description, xacro)
@@ -2,13 +2,12 @@
 <xacro:macro name="flyer">
 <xacro:include filename="$(env MODELS_DIR)/common/utils.xacro" />
+<xacro:include filename="$(env MODELS_DIR)/common/consts.xacro" />
 <xacro:include filename="$(env MODELS_DIR)/flyer/propeller.xacro" />
 <xacro:include filename="$(env MODELS_DIR)/flyer/sslidar.xacro" />
 <link name="base">
     <visual name="base_visual">
-        <origin  xyz="0 0 ${-robot_side_len/2}" rpy="${pi / 2} 0 ${pi / 2}"/>
+        <origin  xyz="0 ${robot_side_len/2 - 0.01} 0" rpy="0 0 ${pi / 2}"/>
         <geometry>
-            <mesh
-                filename="file:///$(env MODELS_DIR)/flyer/Astro_m.stl"
-            />
+            <mesh filename="file:///$(env MODELS_DIR)/flyer/robot.stl" scale="0.001 0.001 0.001"/>
         </geometry>
         <material name="blue">
@@ -24,11 +23,8 @@
 </link>
 <link name="base_weight">
-    <inertial>
-        <mass value="${robot_mass}" />
-        <inertia ixx="${robot_mass/6}" ixy="0" ixz="0" iyy="${robot_mass/6}" iyz="0" izz="${robot_mass/6}"/>
-    </inertial>
+    <xacro:cuboid_inertia weight="2" a="${robot_side_len}" b="${robot_side_len}" c="${robot_side_len}" />
     <visual name="base_visual">
         <geometry>
-            <sphere radius="0.08"/>
+            <sphere radius="${robot_side_len/2 + 0.03}"/>
             <material name="red">
                 <color rgba="1.0 0 0 1.0"/>
@@ -85,9 +81,9 @@
 <!-- END CAMERA BLOCK-->
 <!-- LIDAR BLOCK-->
-<xacro:sslidar name="front" xyz="${robot_side_len/2} 0 0" rpy="0 0 0"/>
-<xacro:sslidar name="back" xyz="${-robot_side_len/2} 0 0" rpy="0 0 ${pi}"/>
-<xacro:sslidar name="right" xyz="0 ${-robot_side_len/2} 0" rpy="0 0 ${-pi / 2}"/>
-<xacro:sslidar name="left" xyz="0 ${robot_side_len/2} 0" rpy="0 0 ${pi / 2}"/>
-<!-- END LIDAR BLOCk-->
+<xacro:sslidar name="fl" xyz="${robot_side_len/2} ${robot_side_len/2} 0" rpy="0 0 ${pi/4}"/>
+<xacro:sslidar name="bl" xyz="${-robot_side_len/2} ${robot_side_len/2} 0" rpy="0 0 ${-pi/4 - pi}"/>
+<xacro:sslidar name="fr" xyz="${robot_side_len/2} ${-robot_side_len/2} 0" rpy="0 0 ${-pi/4}"/>
+<xacro:sslidar name="br" xyz="${-robot_side_len/2} ${-robot_side_len/2} 0" rpy="0 0 ${pi/4 + pi}"/>
+<!-- END LIDAR BLOCK-->
 <gazebo>
     <plugin
@@ -105,12 +101,13 @@
   </plugin>
 </gazebo>
-<xacro:propeller name="prop_fl" xyz="0.1 0.074 0.015" rpy="0 0 ${pi}"/>
-<xacro:propeller name="prop_fr" xyz="0.1 -0.074 0.015" rpy="0 0 ${pi}"/>
-<xacro:propeller name="prop_bl" xyz="-0.1 0.074 0.015" rpy="0 0 0"/>
-<xacro:propeller name="prop_br" xyz="-0.1 -0.074 0.015" rpy="0 0 0"/>
-<xacro:propeller name="prop_rt" xyz="0.04 -0.1 0.073" rpy="0 0 ${pi/2}"/>
-<xacro:propeller name="prop_rb" xyz="-0.04 -0.1 -0.073" rpy="0 0 ${pi/2}"/>
-<xacro:propeller name="prop_lt" xyz="-0.04 0.1 0.073" rpy="0 0 ${-pi/2}"/>
-<xacro:propeller name="prop_lb" xyz="0.04 0.1 -0.073" rpy="0 0 ${-pi/2}"/>
+<xacro:property name="side_offset" value="0.074" />
+<xacro:propeller name="prop_fl" xyz="0.1 ${side_offset} 0.015" rpy="0 0 ${pi}"/>
+<xacro:propeller name="prop_fr" xyz="0.1 ${-side_offset} 0.015" rpy="0 0 ${pi}"/>
+<xacro:propeller name="prop_bl" xyz="-0.1 ${side_offset} 0.015" rpy="0 0 0"/>
+<xacro:propeller name="prop_br" xyz="-0.1 ${-side_offset} 0.015" rpy="0 0 0"/>
+<xacro:propeller name="prop_rt" xyz="0.04 -0.1 ${side_offset}" rpy="0 0 ${pi/2}"/>
+<xacro:propeller name="prop_rb" xyz="-0.04 -0.1 ${-side_offset}" rpy="0 0 ${pi/2}"/>
+<xacro:propeller name="prop_lt" xyz="-0.04 0.1 ${side_offset}" rpy="0 0 ${-pi/2}"/>
+<xacro:propeller name="prop_lb" xyz="0.04 0.1 ${-side_offset}" rpy="0 0 ${-pi/2}"/>
 </xacro:macro>
 </include>

File: models/worlds/stand/stand.sdf.xacro (robot description, xacro)
@@ -1,13 +1,18 @@
 <?xml version="1.0" ?>
 <sdf xmlns:xacro="http://www.ros.org/wiki/xacro" version="1.10">
-<xacro:include filename="$(env MODELS_DIR)/worlds/infinistand/infinistand.xacro" />
 <world name="infinistand_world">
-    <xacro:infinistand_world/>
-    <model name='airstand'>
-        <include>
-             <uri>file:/$(env MODELS_DIR)/platform/full_platform.urdf</uri>
-             <pose>0.0 0.0 0.3275 0.0 0 0.0</pose>
-        </include>
-    </model>
+<xacro:include filename="$(env MODELS_DIR)/common/simple_light.xacro" />
+<xacro:include filename="$(env MODELS_DIR)/common/plugins.xacro" />
+<xacro:include filename="$(env MODELS_DIR)/objects/glass.xacro" />
+<model name="Glass">
+    <static>true</static>
+    <xacro:glass_plate z="-0.01" w="100" l="100" thickness="0.02"/>
+</model>
+<model name='airstand'>
+    <include>
+            <uri>file:/$(env MODELS_DIR)/objects/platform/full_platform.urdf</uri>
+            <pose>0.0 0.0 0.3275 0.0 0 0.0</pose>
+    </include>
+</model>
 </world>
 </sdf>
