Commit message: wip

File: models/common/consts.xacro (robot description, xacro)
@@ -1,4 +1,4 @@
 <include xmlns:xacro="http://www.ros.org/wiki/xacro">
 <xacro:property name="base_height" value="0.655" />
-<xacro:property name="robot_side_len" value="0.22" />
+<xacro:property name="robot_side_len" value="0.24" />
 </include>

File: models/flyer/flyer.xacro (robot description, xacro)
@@ -5,7 +5,8 @@
 <xacro:include filename="$(env MODELS_DIR)/flyer/propeller.xacro" />
 <xacro:include filename="$(env MODELS_DIR)/flyer/sslidar.xacro" />
+<xacro:property name="side_offset" value="0.07" />
 <link name="base">
     <visual name="base_visual">
-        <origin  xyz="0 ${robot_side_len/2 - 0.01} 0" rpy="0 0 ${pi / 2}"/>
+        <origin  xyz="0 ${robot_side_len/2 - 0.02} 0" rpy="0 0 ${pi / 2}"/>
         <geometry>
             <mesh filename="file:///$(env MODELS_DIR)/flyer/robot.stl" scale="0.001 0.001 0.001"/>
@@ -58,5 +59,5 @@
     <parent link="base"/>
     <child link="camera"/>
-    <origin xyz="0 0 ${robot_side_len/2}"/>
+    <origin xyz="${robot_side_len/2 + 0.005} 0 ${side_offset}"/>
 </joint>
 <gazebo reference="camera">
@@ -99,15 +100,22 @@
         <joint_name>prop_lt_joint</joint_name>
         <joint_name>prop_lb_joint</joint_name>
+        <joint_name>prop_ul_joint</joint_name>
+        <joint_name>prop_ur_joint</joint_name>
+        <joint_name>prop_dl_joint</joint_name>
+        <joint_name>prop_dr_joint</joint_name>
   </plugin>
 </gazebo>
-<xacro:property name="side_offset" value="0.074" />
-<xacro:propeller name="prop_fl" xyz="0.1 ${side_offset} 0.015" rpy="0 0 ${pi}"/>
-<xacro:propeller name="prop_fr" xyz="0.1 ${-side_offset} 0.015" rpy="0 0 ${pi}"/>
-<xacro:propeller name="prop_bl" xyz="-0.1 ${side_offset} 0.015" rpy="0 0 0"/>
-<xacro:propeller name="prop_br" xyz="-0.1 ${-side_offset} 0.015" rpy="0 0 0"/>
-<xacro:propeller name="prop_rt" xyz="0.04 -0.1 ${side_offset}" rpy="0 0 ${pi/2}"/>
-<xacro:propeller name="prop_rb" xyz="-0.04 -0.1 ${-side_offset}" rpy="0 0 ${pi/2}"/>
-<xacro:propeller name="prop_lt" xyz="-0.04 0.1 ${side_offset}" rpy="0 0 ${-pi/2}"/>
-<xacro:propeller name="prop_lb" xyz="0.04 0.1 ${-side_offset}" rpy="0 0 ${-pi/2}"/>
+<xacro:propeller name="prop_fl" xyz="${robot_side_len/2} ${side_offset} ${side_offset}" rpy="0 0 ${pi}"/>
+<xacro:propeller name="prop_fr" xyz="${robot_side_len/2} ${-side_offset} ${-side_offset}" rpy="0 0 ${pi}"/>
+<xacro:propeller name="prop_bl" xyz="${-robot_side_len/2} ${side_offset} ${-side_offset}" rpy="0 0 0"/>
+<xacro:propeller name="prop_br" xyz="${-robot_side_len/2} ${-side_offset} ${side_offset}" rpy="0 0 0"/>
+<xacro:propeller name="prop_rt" xyz="${side_offset} ${-robot_side_len/2} ${side_offset}" rpy="0 0 ${pi/2}"/>
+<xacro:propeller name="prop_rb" xyz="${-side_offset} ${-robot_side_len/2} ${-side_offset}" rpy="0 0 ${pi/2}"/>
+<xacro:propeller name="prop_lt" xyz="${-side_offset} ${robot_side_len/2} ${side_offset}" rpy="0 0 ${-pi/2}"/>
+<xacro:propeller name="prop_lb" xyz="${side_offset} ${robot_side_len/2} ${-side_offset}" rpy="0 0 ${-pi/2}"/>
+<xacro:propeller name="prop_ul" xyz="${-side_offset} ${side_offset} ${robot_side_len/2}" rpy="0 ${pi/2} 0"/>
+<xacro:propeller name="prop_ur" xyz="${side_offset} ${-side_offset} ${robot_side_len/2}" rpy="0 ${pi/2} 0"/>
+<xacro:propeller name="prop_dl" xyz="${side_offset} ${side_offset} ${-robot_side_len/2}" rpy="0 ${-pi/2} 0"/>
+<xacro:propeller name="prop_dr" xyz="${-side_offset} ${-side_offset} ${-robot_side_len/2}" rpy="0 ${-pi/2} 0"/>
 </xacro:macro>
 </include>

File: models/worlds/wall/wall.sdf.xacro (robot description, xacro)
@@ -5,13 +5,9 @@
 <xacro:include filename="$(env MODELS_DIR)/common/plugins.xacro" />
 <xacro:include filename="$(env MODELS_DIR)/common/consts.xacro" />
-<xacro:include filename="$(env MODELS_DIR)/objects/glass.xacro" />
-<model name="Glass">
-    <static>true</static>
-    <xacro:glass_plate z="-0.01" w="100" l="100" thickness="0.02"/>
-</model>
-<model name='airstand'>
+<gravity>0 0 0</gravity>
+<model name='flyer'>
     <include>
-        <uri>file:/$(env MODELS_DIR)/objects/platform/full_platform.urdf</uri>
-        <pose>0.0 0.0 ${robot_side_len/2 + base_height/2} 0.0 0 0.0</pose>
+            <uri>file:/$(env MODELS_DIR)/flyer/flyer.urdf</uri>
+            <pose>0.0 0.0 ${robot_side_len/2} 0.0 0 0.0</pose>
     </include>
 </model>

Commit message: add support for multiple robot types

File: models/common/consts.xacro (robot description, xacro)
@@ -1,4 +1,5 @@
 <include xmlns:xacro="http://www.ros.org/wiki/xacro">
 <xacro:property name="base_height" value="0.655" />
-<xacro:property name="robot_side_len" value="0.24" />
+<xacro:property name="robot_side_len_full" value="0.24" />
+<xacro:property name="robot_side_len_proto" value="0.24" />
 </include>

File: models/flyers/full/flyer.urdf.xacro (robot description, xacro)
@@ -1,5 +1,5 @@
 <?xml version="1.0"?>
 <robot name="flyer" xmlns:xacro="http://www.ros.org/wiki/xacro">
-<xacro:include filename="$(env MODELS_DIR)/flyer/flyer.xacro" />
+<xacro:include filename="./flyer.xacro" />
 <xacro:flyer/>
 </robot>

File: models/flyers/full/flyer.xacro (robot description, xacro)
@@ -3,6 +3,7 @@
 <xacro:include filename="$(env MODELS_DIR)/common/utils.xacro" />
 <xacro:include filename="$(env MODELS_DIR)/common/consts.xacro" />
-<xacro:include filename="$(env MODELS_DIR)/flyer/propeller.xacro" />
-<xacro:include filename="$(env MODELS_DIR)/flyer/sslidar.xacro" />
+<xacro:include filename="$(env MODELS_DIR)/flyers/propeller.xacro" />
+<xacro:include filename="$(env MODELS_DIR)/flyers/sslidar.xacro" />
+<xacro:property name="robot_side_len" value="${robot_side_len_full}" />
 <xacro:property name="side_offset" value="0.07" />
 <link name="base">
@@ -10,5 +11,5 @@
         <origin  xyz="0 ${robot_side_len/2 - 0.02} 0" rpy="0 0 ${pi / 2}"/>
         <geometry>
-            <mesh filename="file:///$(env MODELS_DIR)/flyer/robot.stl" scale="0.001 0.001 0.001"/>
+            <mesh filename="file:///$(env MODELS_DIR)/flyers/full/robot.stl" scale="0.001 0.001 0.001"/>
         </geometry>
         <material name="blue">

File: models/objects/platform/full_platform.urdf.xacro (robot description, xacro)
@@ -2,12 +2,12 @@
 <robot name="airstand" xmlns:xacro="http://www.ros.org/wiki/xacro">
 <xacro:include filename="$(env MODELS_DIR)/common/consts.xacro" />
-<xacro:include filename="$(env MODELS_DIR)/flyer/flyer.xacro" />
+<xacro:include filename="$(env MODELS_DIR)/flyers/proto/proto.xacro" />
 <xacro:include filename="./platform.xacro" />
 <xacro:platform/>
-<xacro:flyer/>
-<joint name="platform_flyer_joint" type="fixed">
+<xacro:proto/>
+<joint name="platform_proto_joint" type="fixed">
     <parent link="platform"/>
     <child link="base"/>
-    <origin xyz="0 0 ${robot_side_len/2 + base_height/2}"/>
+    <origin xyz="0 0 ${robot_side_len_proto/2 + base_height/2}"/>
 </joint>
 </robot>

File: models/objects/platform/platform.urdf.xacro (robot description, xacro)
@@ -2,5 +2,4 @@
 <robot name="platform" xmlns:xacro="http://www.ros.org/wiki/xacro">
 <xacro:include filename="$(env MODELS_DIR)/common/utils.xacro" />
-<xacro:include filename="$(env MODELS_DIR)/flyer/flyer.xacro" />
 <xacro:include filename="./platform.xacro" />
 <xacro:platform/>

File: models/worlds/stand/stand.sdf.xacro (robot description, xacro)
@@ -13,5 +13,5 @@
     <include>
         <uri>file:/$(env MODELS_DIR)/objects/platform/full_platform.urdf</uri>
-        <pose>0.0 0.0 ${robot_side_len/2 + base_height/2} 0.0 0 0.0</pose>
+        <pose>0.0 0.0 ${base_height/2 + 0.01} 0.0 0 0.0</pose>
     </include>
 </model>

File: models/worlds/wall/wall.sdf.xacro (robot description, xacro)
@@ -8,6 +8,6 @@
 <model name='flyer'>
     <include>
-            <uri>file:/$(env MODELS_DIR)/flyer/flyer.urdf</uri>
-            <pose>0.0 0.0 ${robot_side_len/2} 0.0 0 0.0</pose>
+            <uri>file:/$(env MODELS_DIR)/flyers/full/flyer.urdf</uri>
+            <pose>0.0 0.0 ${robot_side_len_full/2} 0.0 0 0.0</pose>
     </include>
 </model>
