Commit message: fix gz<->ros integration and odom

File: models/common/plugins.xacro (robot description, xacro)
@@ -21,5 +21,5 @@
 <plugin filename="gz-sim-sensors-system"
         name="gz::sim::systems::Sensors">
-    <render_engine>ogre2</render_engine>
+    <render_engine>ogre</render_engine>
 </plugin>
 </include>

File: models/flyers/full/flyer.xacro (robot description, xacro)
@@ -11,5 +11,5 @@
         <origin  xyz="0 ${robot_side_len/2 - 0.02} 0" rpy="0 0 ${pi / 2}"/>
         <geometry>
-            <mesh filename="file:///$(env MODELS_DIR)/flyers/full/robot.stl" scale="0.001 0.001 0.001"/>
+            <mesh filename="file:///$(env MODELS_DIR)/flyers/full/simplify_robot.stl" scale="0.001 0.001 0.001"/>
         </geometry>
         <material name="blue">
@@ -60,9 +60,10 @@
         filename="gz-sim-odometry-publisher-system"
         name="gz::sim::systems::OdometryPublisher">
-        <odom_frame>/ground-truth/odom</odom_frame>
+        <odom_frame>/ground_truth/odom</odom_frame>
         <robot_base_frame>base</robot_base_frame>
         <odom_publish_frequency>20</odom_publish_frequency>
-        <odom_topic>/ground-truth/odom</odom_topic>
+        <odom_topic>/ground_truth/odom</odom_topic>
         <tf_topic>tf</tf_topic>
+        <dimensions>3</dimensions>
   </plugin>
 </gazebo>
