Commit message: add iss floor

File: models/common/simple_light.xacro (robot description, xacro)
@@ -11,5 +11,5 @@
         <quadratic>0.001</quadratic>
     </attenuation>
-    <direction>-0.5 0.1 -0.9</direction>
+    <direction>1 0 -1</direction>
 </light>
 <scene>

File: models/objects/wall/panel_utils.xacro (robot description, xacro)
@@ -1,30 +1,3 @@
-<?xml version="1.0" ?>
-<sdf xmlns:xacro="http://www.ros.org/wiki/xacro" version="1.10">
-<model name="panel_105">
-<pose>0 0 0 0 0 0</pose>
-<static>true</static>
-<link name="panel_105">
-    <self_collide>false</self_collide>
-    <collision name="panel_105_collision">
-        <geometry>
-            <box>
-                <size>1 1 1</size>
-            </box>
-        </geometry>
-    </collision>
-    <visual name="panel_105_visual">
-        <geometry>
-            <mesh>
-                <uri>file:/$(env MODELS_DIR)/objects/wall/100-panels/105.stl</uri>
-                <scale>1 1 1</scale>
-            </mesh>
-        </geometry>
-        <material>
-            <ambient>0 0.3 0 1</ambient>
-            <diffuse>0 0.4 0 1</diffuse>
-            <specular>0.3 0.6 0.3 1</specular>
-        </material>
-    </visual>
-</link>
+<include xmlns:xacro="http://www.ros.org/wiki/xacro">
 <xacro:macro name="simple_obj" params="name reference pose model">
     <link name="${name}">
@@ -66,12 +39,4 @@
     />
 </xacro:macro>
-<xacro:lock name="lock_1" pose="0.053 -0.434 0.0197 0 0  1.57" reference="panel_105"/>
-<xacro:lock name="lock_2" pose="0.053  0.434 0.0197 0 0  1.57" reference="panel_105"/>
-<xacro:lock name="lock_3" pose="0.415 -0.434 0.0197 0 0 -1.57" reference="panel_105"/>
-<xacro:lock name="lock_4" pose="0.415  0.434 0.0197 0 0 -1.57" reference="panel_105"/>
-<xacro:locker name="locker_1" pose="0.0575 -0.250 0.0197 0 0 -3.14" reference="panel_105"/>
-<xacro:locker name="locker_2" pose="0.0575  0.250 0.0197 0 0 -3.14" reference="panel_105"/>
-<xacro:locker name="locker_3" pose="0.4105 -0.250 0.0197 0 0  3.14" reference="panel_105"/>
-<xacro:locker name="locker_4" pose="0.4105  0.250 0.0197 0 0  3.14" reference="panel_105"/>
 <xacro:macro name="simple_shield" params="name reference size pose img">
     <link name="${name}">
@@ -101,5 +66,5 @@
     </joint>
 </xacro:macro>
-<xacro:macro name="shield50x80" params="name reference pose">
+<xacro:macro name="shield50x80" params="name:='shield50x80' reference pose img_ref_wall">
     <xacro:simple_shield
         name="${name}"
@@ -107,8 +72,8 @@
         pose="${pose}"
         reference="${reference}"
-        img="file:/$(env MODELS_DIR)/objects/wall/100-panels/105-50x80.png"
+        img="file:/$(env MODELS_DIR)/objects/wall/${img_ref_wall}"
     />
 </xacro:macro>
-<xacro:macro name="shield145x30" params="name reference pose">
+<xacro:macro name="shield145x30" params="name:='shield145x30' reference pose img_ref_wall">
     <xacro:simple_shield
         name="${name}"
@@ -116,9 +81,36 @@
         pose="${pose}"
         reference="${reference}"
-        img="file:/$(env MODELS_DIR)/objects/wall/100-panels/105-145x30.png"
+        img="file:/$(env MODELS_DIR)/objects/wall/${img_ref_wall}"
     />
 </xacro:macro>
-<xacro:shield50x80 name="shield50x80" pose="0.05 0 0.0198 0 0 1.57" reference="panel_105"/>
-<xacro:shield145x30 name="shield145x30" pose="0.139 0 0.0198 0 0 1.57" reference="panel_105"/>
-</model>
-</sdf>
+<xacro:macro name="shield100x30" params="name:='shield100x30' reference pose img_ref_wall">
+    <xacro:simple_shield
+        name="${name}"
+        size="0.1 0.03"
+        pose="${pose}"
+        reference="${reference}"
+        img="file:/$(env MODELS_DIR)/objects/wall/${img_ref_wall}"
+    />
+</xacro:macro>
+<xacro:macro name="panel" params="name size model_ref_wall *material">
+    <link name="${name}">
+        <self_collide>false</self_collide>
+        <collision name="${name}_collision">
+            <geometry>
+                <box>
+                    <size>${size}</size>
+                </box>
+            </geometry>
+        </collision>
+        <visual name="${name}_visual">
+            <geometry>
+                <mesh>
+                    <uri>file:/$(env MODELS_DIR)/objects/wall/${model_ref_wall}</uri>
+                    <scale>1 1 1</scale>
+                </mesh>
+            </geometry>
+            <xacro:insert_block name="material" />
+        </visual>
+    </link>
+</xacro:macro>
+</include>

File: models/worlds/wall/wall.sdf.xacro (robot description, xacro)
@@ -12,8 +12,21 @@
     </include>
 </model>
-<model name='wall'>
+<model name='floor'>
+    <pose>1 0 2 0 ${pi / 2} ${pi}</pose>
     <include>
-            <uri>file:/$(env MODELS_DIR)/objects/wall/100-panels</uri>
-            <pose>1 0 0 0 0 0</pose>
+        <uri>file:/$(env MODELS_DIR)/objects/wall/100-panels/105</uri>
+        <pose>0 0 0 0 0 0</pose>
+    </include>
+    <include>
+        <uri>file:/$(env MODELS_DIR)/objects/wall/100-panels/106</uri>
+        <pose>0.503 0 0 0 0 0</pose>
+    </include>
+    <include>
+        <uri>file:/$(env MODELS_DIR)/objects/wall/100-panels/107</uri>
+        <pose>1.073 0 0 0 0 0</pose>
+    </include>
+    <include>
+        <uri>file:/$(env MODELS_DIR)/objects/wall/100-panels/108</uri>
+        <pose>1.723 0 0 0 0 0</pose>
     </include>
 </model>
