Commit message: update wall world

File: models/flyers/full/flyer.xacro (robot description, xacro)
@@ -26,4 +26,5 @@
 <link name="base_weight">
     <xacro:cuboid_inertia weight="2" a="${robot_side_len}" b="${robot_side_len}" c="${robot_side_len}" />
+    <!--
     <visual name="base_visual">
         <geometry>
@@ -34,4 +35,5 @@
         </geometry>
     </visual>
+    -->
 </link>
 <joint name="base_weight_joint" type="fixed">
@@ -81,6 +83,6 @@
             <horizontal_fov>1.047</horizontal_fov>
             <image>
-                <width>320</width>
-                <height>240</height>
+                <width>640</width>
+                <height>480</height>
             </image>
             <clip>

File: models/worlds/wall/wall.sdf.xacro (robot description, xacro)
@@ -13,5 +13,30 @@
 </model>
 <model name='floor'>
+    <static>true</static>
     <pose>1 0 2 0 ${pi / 2} ${pi}</pose>
+    <link name="backpanel">
+        <pose>0 0 -0.1 0 0 0</pose>
+        <self_collide>false</self_collide>
+        <visual name="backpanel_visual">
+            <geometry>
+                <box>
+                    <size>7 2 0.2</size>
+                </box>
+            </geometry>
+            <material>
+                <script>
+                    <uri>file://media/materials/scripts/gazebo.material</uri>
+                    <name>Gazebo/Grey</name>
+                </script>
+            </material>
+        </visual>
+        <collision name="backpanel_collision">
+            <geometry>
+                <box>
+                    <size>7 2 0.2</size>
+                </box>
+            </geometry>
+        </collision>
+    </link>
     <include>
         <uri>file:/$(env MODELS_DIR)/objects/wall/100-panels/105</uri>
